Commit message: added a cylinder in gazebo for bin

File: install/robot_description/share/robot_description/urdf/camera.urdf.xacro (robot description, xacro)
@@ -30,5 +30,34 @@
         <parent link="dummy_root_link"/>
         <child link="camera_link"/>
-        <origin xyz="0.0 1.0 0.5" rpy="0 0 -1.57"/>  <!-- Adjust this to position the camera -->
+        <origin xyz="0.5 0.7 0.5" rpy="0 0 -3.14"/>  <!-- Adjust this to position the camera -->
+    </joint>
+    <!-- Cylinder at a distance of 1.5 along the x-axis from the camera -->
+    <link name="cylinder_link">
+        <visual>
+            <origin xyz="0.5 0.0 0.0" rpy="0 0 0"/>  <!-- Positioned 1.5 units in the x direction -->
+            <geometry>
+                <cylinder radius="0.2" length="0.5"/>  <!-- Cylinder shape with radius and length -->
+            </geometry>
+            <material name="Red">
+                <color rgba="1.0 0.0 0.0 1.0"/>
+            </material>
+        </visual>
+        <collision>
+            <origin xyz="1.5 0.0 0.0" rpy="0 0 0"/>
+            <geometry>
+                <cylinder radius="0.05" length="0.2"/>
+            </geometry>
+        </collision>
+        <inertial>
+            <origin xyz="0 0 0"/>
+            <mass value="0.2"/>  <!-- Adjust mass based on size -->
+            <inertia ixx="0.0001" ixy="0" ixz="0" iyy="0.0001" iyz="0" izz="0.0001"/>
+        </inertial>
+    </link>
+    <!-- Fixed joint connecting camera link to the cylinder link -->
+    <joint name="camera_to_cylinder_joint" type="fixed">
+        <parent link="camera_link"/>
+        <child link="cylinder_link"/>
+        <origin xyz="0.5 0.0 0.0" rpy="0 0 0"/>
     </joint>
     <!-- Gazebo sensor configuration -->
@@ -46,4 +75,9 @@
                     <far>300</far>
                 </clip>
+                <noise>
+                    <type>gaussian</type>
+                    <mean>0.0</mean>
+                    <stddev>0.007</stddev>
+                </noise>
             </camera>
             <always_on>true</always_on>

File: install/robot_description/share/robot_description/urdf/robot.urdf.xacro (robot description, xacro)
@@ -263,8 +263,31 @@
         </xacro:cylinder_inertial>
     </link>
-    <!-- <joint name="camera_joint" type="fixed">
+    <!-- <joint name="checkered_box_joint" type="fixed">
         <parent link="wrist_3_link" />
-        <child link="camera_link" />
+        <child link="checkered_box_link" />
         <origin xyz="0.0 0.09 0.0025" rpy="0.0 0.0 ${pi/2}" />
-    </joint> -->
+    </joint>
+    <link name="checkered_box_link">
+        <visual>
+            <scale>0.5 0.5 0.5</scale>  This scales the mesh by 50%
+            <geometry>
+                <box size="0.025 0.25 0.25"/>
+            </geometry>
+            <material name="Black">
+                <color rgba="0.0 0.0 0.0 1.0"/>
+            </material>
+        </visual>
+        <collision>
+            <geometry>
+                <box size="0.001 0.001 0.001"/>
+            </geometry>
+        </collision>
+        <inertial>
+            <origin xyz="0.0 0.0 0.0" rpy="0 0 0"/>
+            <mass value="0.1"/>
+            <inertia ixx="0.0001" ixy="0.0" ixz="0.0"
+                     iyy="0.0001" iyz="0.0"
+                     izz="0.0001"/>
+        </inertial>
+    </link> -->
 </robot>

File: src/robot_description/urdf/camera.urdf.xacro (robot description, xacro)
@@ -30,5 +30,34 @@
         <parent link="dummy_root_link"/>
         <child link="camera_link"/>
-        <origin xyz="0.0 1.5 0.5" rpy="0 0 -1.57"/>  <!-- Adjust this to position the camera -->
+        <origin xyz="0.5 0.7 0.5" rpy="0 0 -3.14"/>  <!-- Adjust this to position the camera -->
+    </joint>
+    <!-- Cylinder at a distance of 1.5 along the x-axis from the camera -->
+    <link name="cylinder_link">
+        <visual>
+            <origin xyz="0.5 0.0 0.0" rpy="0 0 0"/>  <!-- Positioned 1.5 units in the x direction -->
+            <geometry>
+                <cylinder radius="0.2" length="0.5"/>  <!-- Cylinder shape with radius and length -->
+            </geometry>
+            <material name="Red">
+                <color rgba="1.0 0.0 0.0 1.0"/>
+            </material>
+        </visual>
+        <collision>
+            <origin xyz="1.5 0.0 0.0" rpy="0 0 0"/>
+            <geometry>
+                <cylinder radius="0.05" length="0.2"/>
+            </geometry>
+        </collision>
+        <inertial>
+            <origin xyz="0 0 0"/>
+            <mass value="0.2"/>  <!-- Adjust mass based on size -->
+            <inertia ixx="0.0001" ixy="0" ixz="0" iyy="0.0001" iyz="0" izz="0.0001"/>
+        </inertial>
+    </link>
+    <!-- Fixed joint connecting camera link to the cylinder link -->
+    <joint name="camera_to_cylinder_joint" type="fixed">
+        <parent link="camera_link"/>
+        <child link="cylinder_link"/>
+        <origin xyz="0.5 0.0 0.0" rpy="0 0 0"/>
     </joint>
     <!-- Gazebo sensor configuration -->
@@ -46,4 +75,9 @@
                     <far>300</far>
                 </clip>
+                <noise>
+                    <type>gaussian</type>
+                    <mean>0.0</mean>
+                    <stddev>0.007</stddev>
+                </noise>
             </camera>
             <always_on>true</always_on>

File: src/robot_description/urdf/robot.urdf.xacro (robot description, xacro)
@@ -263,5 +263,5 @@
         </xacro:cylinder_inertial>
     </link>
-    <joint name="checkered_box_joint" type="fixed">
+    <!-- <joint name="checkered_box_joint" type="fixed">
         <parent link="wrist_3_link" />
         <child link="checkered_box_link" />
@@ -270,7 +270,4 @@
     <link name="checkered_box_link">
         <visual>
-            <!-- <geometry>
-                <mesh filename="package://robot_description/meshes/checkered_box.dae" />
-            </geometry> -->
             <scale>0.5 0.5 0.5</scale>  This scales the mesh by 50%
             <geometry>
@@ -293,4 +290,4 @@
                      izz="0.0001"/>
         </inertial>
-    </link>
+    </link> -->
 </robot>
