Commit message: till coding part 1

File: install/robot_description/share/robot_description/urdf/robot.urdf.xacro (robot description, xacro)
@@ -6,5 +6,5 @@
     <xacro:include filename="$(find robot_description)/urdf/robot_gazebo.xacro" />
     <!-- Include ros2_control Plugins -->
-    <!-- <xacro:include filename="$(find robot_description)/urdf/robot_ros2_control.xacro" /> -->
+    <xacro:include filename="$(find robot_description)/urdf/robot_ros2_control.xacro" />
     <!-- Useful XACRO Variables (Properties) -->
   <!-- Inertia parameters -->
@@ -263,5 +263,5 @@
         </xacro:cylinder_inertial>
     </link>
-    <!-- <joint name="camera_joint" type="fixed">
+    <joint name="camera_joint" type="fixed">
         <parent link="wrist_3_link" />
         <child link="camera_link" />
@@ -290,5 +290,5 @@
         </inertial>
     </link>
-    <gazebo reference="camera_link">
+    <!-- <gazebo reference="camera_link">
         <sensor type="camera" name="robot_camera">
             <update_rate>30.0</update_rate>

File: install/robot_description/share/robot_description/urdf/robot_gazebo.xacro (robot description, xacro)
@@ -1,7 +1,7 @@
 <?xml version="1.0"?>
-<robot xmlns:xacro="http://www.ros.org/wiki/xacro" name="cobot">
+<robot xmlns:xacro="http://www.ros.org/wiki/xacro" name="crobot">
   <gazebo>
     <plugin filename="gz_ros2_control-system" name="gz_ros2_control::GazeboSimROS2ControlPlugin">
-        <!-- <parameters>$(find cobot_controller)/config/cobot_controllers.yaml</parameters> -->
+        <parameters>$(find robot_controller)/config/ros2_controllers.yaml</parameters>
     </plugin>
   </gazebo>

Commit message: camera sensor plugin added and working

File: install/robot_description/share/robot_description/urdf/robot.urdf.xacro (robot description, xacro)
@@ -266,10 +266,11 @@
         <parent link="wrist_3_link" />
         <child link="camera_link" />
-        <origin xyz="0.0 0.065 0.06" rpy="0.0 0.0 0.0" />
+        <!-- <origin xyz="0.0 0.065 0.06" rpy="0.0 0.0 0.0" /> -->
+        <origin xyz="0.0 0.065 0.06" rpy="0.0 0.0 ${pi/2}" />
     </joint>
     <link name="camera_link">
         <visual>
             <geometry>
-                <box size="0.05 0.025 0.05"/>
+                <box size="0.025 0.05 0.05"/>
             </geometry>
             <material name="Green">
@@ -290,6 +291,26 @@
         </inertial>
     </link>
-    <!-- <gazebo reference="camera_link">
-        <sensor type="camera" name="robot_camera">
+    <gazebo reference="camera_link">
+        <sensor type="camera" name="camera">
+            <camera>
+                <horizontal_fov>1.3962634</horizontal_fov>
+                <image>
+                    <width>640</width>
+                    <height>480</height>
+                    <format>R8G8B8</format>
+                </image>
+                <clip>
+                    <near>0.02</near>
+                    <far>300</far>
+                </clip>
+            </camera>
+            <always_on>true</always_on>
+            <update_rate>30</update_rate>
+            <topic>camera/image_raw</topic>
+            <plugin filename="libignition-gazebo-sensors-system.so" name="ignition::gazebo::systems::Sensors">
+                <render_engine>ogre2</render_engine>
+            </plugin>
+        </sensor>
+        <!-- <sensor type="camera" name="robot_camera">
             <update_rate>30.0</update_rate>
             <camera name="head">
@@ -313,6 +334,7 @@
                 <alwaysOn>true</alwaysOn>
                 <visualize>true</visualize>
+                <image_transport>raw</image_transport>
                 <updateRate>30.0</updateRate>
-                <cameraName>CB/camera</cameraName>
+                <cameraName>camera</cameraName>
                 <imageTopicName>image_raw</imageTopicName>
                 <cameraInfoTopicName>camera_info</cameraInfoTopicName>
@@ -325,5 +347,5 @@
                 <distortionT2>0.0</distortionT2>
             </plugin>
-        </sensor>
-    </gazebo>  -->
+        </sensor> -->
+    </gazebo>
 </robot>

Commit message: implemented camera pose computation with forward kinematics

File: install/robot_description/share/robot_description/urdf/robot.urdf.xacro (robot description, xacro)
@@ -267,5 +267,5 @@
         <child link="camera_link" />
         <!-- <origin xyz="0.0 0.065 0.06" rpy="0.0 0.0 0.0" /> -->
-        <origin xyz="0.0 0.065 0.06" rpy="0.0 0.0 ${pi/2}" />
+        <origin xyz="0.0 0.09 0.0025" rpy="0.0 0.0 ${pi/2}" />
     </joint>
     <link name="camera_link">

Commit message: camera and robot seperate spawn

File: install/robot_description/share/robot_description/urdf/robot.urdf.xacro (robot description, xacro)
@@ -263,89 +263,8 @@
         </xacro:cylinder_inertial>
     </link>
-    <joint name="camera_joint" type="fixed">
+    <!-- <joint name="camera_joint" type="fixed">
         <parent link="wrist_3_link" />
         <child link="camera_link" />
-        <!-- <origin xyz="0.0 0.065 0.06" rpy="0.0 0.0 0.0" /> -->
         <origin xyz="0.0 0.09 0.0025" rpy="0.0 0.0 ${pi/2}" />
-    </joint>
-    <link name="camera_link">
-        <visual>
-            <geometry>
-                <box size="0.025 0.05 0.05"/>
-            </geometry>
-            <material name="Green">
-                <color rgba="0.0 1.0 0.0 1.0"/>
-            </material>
-        </visual>
-        <collision>
-            <geometry>
-                <box size="0.001 0.001 0.001"/>
-            </geometry>
-        </collision>
-        <inertial>
-            <origin xyz="0.0 0.0 0.0" rpy="0 0 0"/>
-            <mass value="0.1"/>
-            <inertia ixx="0.0001" ixy="0.0" ixz="0.0"
-                     iyy="0.0001" iyz="0.0"
-                     izz="0.0001"/>
-        </inertial>
-    </link>
-    <gazebo reference="camera_link">
-        <sensor type="camera" name="camera">
-            <camera>
-                <horizontal_fov>1.3962634</horizontal_fov>
-                <image>
-                    <width>640</width>
-                    <height>480</height>
-                    <format>R8G8B8</format>
-                </image>
-                <clip>
-                    <near>0.02</near>
-                    <far>300</far>
-                </clip>
-            </camera>
-            <always_on>true</always_on>
-            <update_rate>30</update_rate>
-            <topic>camera/image_raw</topic>
-            <plugin filename="libignition-gazebo-sensors-system.so" name="ignition::gazebo::systems::Sensors">
-                <render_engine>ogre2</render_engine>
-            </plugin>
-        </sensor>
-        <!-- <sensor type="camera" name="robot_camera">
-            <update_rate>30.0</update_rate>
-            <camera name="head">
-                <horizontal_fov>1.3962634</horizontal_fov>
-                <image>
-                    <width>640</width>
-                    <height>480</height>
-                    <format>R8G8B8</format>
-                </image>
-                <clip>
-                    <near>0.02</near>
-                    <far>300</far>
-                </clip>
-                <noise>
-                    <type>gaussian</type>
-                    <mean>0.0</mean>
-                    <stddev>0.007</stddev>
-                </noise>
-            </camera>
-            <plugin name="camera_controller" filename="libgazebo_ros_camera.so">
-                <alwaysOn>true</alwaysOn>
-                <visualize>true</visualize>
-                <image_transport>raw</image_transport>
-                <updateRate>30.0</updateRate>
-                <cameraName>camera</cameraName>
-                <imageTopicName>image_raw</imageTopicName>
-                <cameraInfoTopicName>camera_info</cameraInfoTopicName>
-                <frameName>camera_link</frameName>
-                <hackBaseline>0.07</hackBaseline>
-                <distortionK1>0.0</distortionK1>
-                <distortionK2>0.0</distortionK2>
-                <distortionK3>0.0</distortionK3>
-                <distortionT1>0.0</distortionT1>
-                <distortionT2>0.0</distortionT2>
-            </plugin>
-        </sensor> -->
-    </gazebo>
+    </joint> -->
 </robot>

Commit message: add camera 3d pose calib script

File: install/robot_description/share/robot_description/urdf/robot.urdf.xacro (robot description, xacro)
@@ -263,5 +263,5 @@
         </xacro:cylinder_inertial>
     </link>
-    <!-- <joint name="checkered_box_joint" type="fixed">
+    <joint name="checkered_box_joint" type="fixed">
         <parent link="wrist_3_link" />
         <child link="checkered_box_link" />
@@ -270,5 +270,4 @@
     <link name="checkered_box_link">
         <visual>
-            <scale>0.5 0.5 0.5</scale>  This scales the mesh by 50%
             <geometry>
                 <box size="0.025 0.25 0.25"/>
@@ -290,4 +289,4 @@
                      izz="0.0001"/>
         </inertial>
-    </link> -->
+    </link>
 </robot>
