Commit message: added calib target to robot

File: src/robot_description/urdf/robot.urdf.xacro (robot description, xacro)
@@ -263,8 +263,34 @@
         </xacro:cylinder_inertial>
     </link>
-    <!-- <joint name="camera_joint" type="fixed">
+    <joint name="checkered_box_joint" type="fixed">
         <parent link="wrist_3_link" />
-        <child link="camera_link" />
+        <child link="checkered_box_link" />
         <origin xyz="0.0 0.09 0.0025" rpy="0.0 0.0 ${pi/2}" />
-    </joint> -->
+    </joint>
+    <link name="checkered_box_link">
+        <visual>
+            <!-- <geometry>
+                <mesh filename="package://robot_description/meshes/checkered_box.dae" />
+            </geometry> -->
+            <scale>0.5 0.5 0.5</scale>  This scales the mesh by 50%
+            <geometry>
+                <box size="0.025 0.25 0.25"/>
+            </geometry>
+            <material name="Black">
+                <color rgba="0.0 0.0 0.0 1.0"/>
+            </material>
+        </visual>
+        <collision>
+            <geometry>
+                <box size="0.001 0.001 0.001"/>
+            </geometry>
+        </collision>
+        <inertial>
+            <origin xyz="0.0 0.0 0.0" rpy="0 0 0"/>
+            <mass value="0.1"/>
+            <inertia ixx="0.0001" ixy="0.0" ixz="0.0"
+                     iyy="0.0001" iyz="0.0"
+                     izz="0.0001"/>
+        </inertial>
+    </link>
 </robot>

Commit message: commented checkered link

File: src/robot_description/urdf/robot.urdf.xacro (robot description, xacro)
@@ -263,5 +263,5 @@
         </xacro:cylinder_inertial>
     </link>
-    <joint name="checkered_box_joint" type="fixed">
+    <!-- <joint name="checkered_box_joint" type="fixed">
         <parent link="wrist_3_link" />
         <child link="checkered_box_link" />
@@ -289,4 +289,4 @@
                      izz="0.0001"/>
         </inertial>
-    </link>
+    </link> -->
 </robot>
